File: hardware_kicad/filament_dryer.kicad_sch (KiCad schematic)
At the start: 98 parts, among them J1 USB_C_Receptacle_USB2.0, J2 H/T Ambient, J3 T Aux, J4 Peristaltic Pump, Q1 NMOS, Q2 NMOS, Q3 NMOS, Q4 NMOS, U1 W25Q128JVS, U2 AMS1117-3.3, U3 RP2040, U4 DS18B20Z, U5 H/T Filament, X1 12MHz Yangxing Tech X322512MS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

Commit message: Ready for second review
Parts:
- removed D1: HEATER_2, LED_SMD:LED_0603_1608Metric, symbol 00_project_library:LED
- removed D2: HEATER_1, LED_SMD:LED_0603_1608Metric, symbol 00_project_library:LED
- removed Q1, Q2: NMOS, Package_TO_SOT_SMD:SOT-23, symbol 00_project_library:NMOS
- removed R11, R7: 470R, Resistor_SMD:R_0402_1005Metric_Pad0.72x0.64mm_HandSolder, symbol 00_project_library:R
- removed R_POWER1_1, R_POWER1_10, R_POWER1_11, R_POWER1_12, R_POWER1_2, R_POWER1_3, R_POWER1_4, R_POWER1_5, R_POWER1_6, R_POWER1_7, R_POWER1_8, R_POWER1_9, R_POWER2_1, R_POWER2_10, R_POWER2_11, R_POWER2_12, R_POWER2_2, R_POWER2_3, R_POWER2_4, R_POWER2_5, R_POWER2_6, R_POWER2_7, R_POWER2_8, R_POWER2_9: 120, Resistor_SMD:R_1206_3216Metric, symbol 00_project_library:R_POWER
- added D10, D11, D8, D9: 1N4148WS, Diode_SMD:D_SOD-323, symbol Diode:1N4148WS
- added JP1, JP2, JP3, JP4: SolderJumper_2_Open, Jumper:SolderJumper-2_P1.3mm_Open_RoundedPad1.0x1.5mm, symbol Jumper:SolderJumper_2_Open
- added NeoC1, NeoC10, NeoC11, NeoC12, NeoC13, NeoC14, NeoC15, NeoC16, NeoC17, NeoC18, NeoC19, NeoC2, NeoC20, NeoC21, NeoC22, NeoC23, NeoC24, NeoC25, NeoC26, NeoC27, NeoC28, NeoC3, NeoC4, NeoC5, NeoC6, NeoC7, NeoC8, NeoC9: 100n, Capacitor_SMD:C_0402_1005Metric_Pad0.74x0.62mm_HandSolder, symbol 00_project_library:C
- added NeoD1, NeoD10, NeoD11, NeoD12, NeoD13, NeoD14, NeoD15, NeoD16, NeoD17, NeoD18, NeoD19, NeoD2, NeoD20, NeoD21, NeoD22, NeoD23, NeoD24, NeoD25, NeoD26, NeoD27, NeoD28, NeoD3, NeoD4, NeoD5, NeoD6, NeoD7, NeoD8, NeoD9: WS2812B-2020, LED_SMD:LED_WS2812B-2020_PLCC4_2.0x2.0mm, symbol 00_project_library:WS2812B-2020
- added Q5, Q6, Q7, Q8: NMOS, Package_TO_SOT_SMD:SOT-23, symbol 00_project_library:NMOS
- added R1, R17, R18, R21: 4K7, Resistor_SMD:R_0402_1005Metric_Pad0.72x0.64mm_HandSolder, symbol 00_project_library:R
- J2, J3, J4: now left out of the parts list
Connections:
- net +3V3: now also Q5.2 (G), Q6.2 (G), Q7.2 (G), Q8.2 (G)
- net +5V: now also NeoC1.1, NeoC10.1, NeoC11.1, NeoC12.1, NeoC13.1, NeoC14.1, NeoC15.1, NeoC16.1, NeoC17.1, NeoC18.1, NeoC19.1, NeoC2.1, NeoC20.1, NeoC21.1, NeoC22.1, NeoC23.1, NeoC24.1, NeoC25.1, NeoC26.1, NeoC27.1, NeoC28.1, NeoC3.1, NeoC4.1, NeoC5.1, NeoC6.1, NeoC7.1, NeoC8.1, NeoC9.1, NeoD1.4 (VDD), NeoD10.4 (VDD), NeoD11.4 (VDD), NeoD12.4 (VDD), NeoD13.4 (VDD), NeoD14.4 (VDD), NeoD15.4 (VDD), NeoD16.4 (VDD), NeoD17.4 (VDD), NeoD18.4 (VDD), NeoD19.4 (VDD), NeoD2.4 (VDD), NeoD20.4 (VDD), NeoD21.4 (VDD), NeoD22.4 (VDD), NeoD23.4 (VDD), NeoD24.4 (VDD), NeoD25.4 (VDD), NeoD26.4 (VDD), NeoD27.4 (VDD), NeoD28.4 (VDD), NeoD3.4 (VDD), NeoD4.4 (VDD), NeoD5.4 (VDD), NeoD6.4 (VDD), NeoD7.4 (VDD), NeoD8.4 (VDD), NeoD9.4 (VDD), R1.1, R17.1, R18.1, R21.1
- net GND: now also NeoC1.2, NeoC10.2, NeoC11.2, NeoC12.2, NeoC13.2, NeoC14.2, NeoC15.2, NeoC16.2, NeoC17.2, NeoC18.2, NeoC19.2, NeoC2.2, NeoC20.2, NeoC21.2, NeoC22.2, NeoC23.2, NeoC24.2, NeoC25.2, NeoC26.2, NeoC27.2, NeoC3.2, NeoC4.2, NeoC5.2, NeoC6.2, NeoC7.2, NeoC8.2, NeoC9.2, NeoD1.2 (GND), NeoD10.2 (GND), NeoD11.2 (GND), NeoD12.2 (GND), NeoD13.2 (GND), NeoD14.2 (GND), NeoD15.2 (GND), NeoD16.2 (GND), NeoD17.2 (GND), NeoD18.2 (GND), NeoD19.2 (GND), NeoD2.2 (GND), NeoD20.2 (GND), NeoD21.2 (GND), NeoD22.2 (GND), NeoD23.2 (GND), NeoD24.2 (GND), NeoD25.2 (GND), NeoD26.2 (GND), NeoD27.2 (GND), NeoD28.2 (GND), NeoD3.2 (GND), NeoD4.2 (GND), NeoD5.2 (GND), NeoD6.2 (GND), NeoD7.2 (GND), NeoD8.2 (GND), NeoD9.2 (GND)
- net GPIO_NP_A: now reaches U3.3 (GPIO1)
- net GPIO_NP_A: now also JP1.1 (A), Q5.3 (S)
- net GPIO_NP_B: now reaches U3.37 (GPIO25)
- net GPIO_NP_B: now also JP2.1 (A), Q6.3 (S)
- net GPIO_NP_C: now reaches U3.4 (GPIO2)
- net GPIO_NP_C: now also JP3.1 (A), Q7.3 (S)
- net T_BOARD_1WIRE: no longer names the net of U3.12 (GPIO9)
- net T_BOARD_1WIRE: no longer U3.2 (GPIO0)
- new net: NeoD19.1 (DOUT), NeoD20.3 (DIN)
- new net: NeoD18.1 (DOUT), NeoD19.3 (DIN)
- new net: NeoD16.1 (DOUT), NeoD17.3 (DIN)
- new net: NeoD15.1 (DOUT), NeoD16.3 (DIN)
- new net: D11.1 (K), NeoD27.3 (DIN), Q8.1 (D), R21.2
- new net: D9.1 (K), NeoD11.3 (DIN), Q6.1 (D), R17.2
- new net: NeoD25.1 (DOUT), NeoD26.3 (DIN)
- new net: NeoD24.1 (DOUT), NeoD25.3 (DIN)
- new net: NeoD23.1 (DOUT), NeoD24.3 (DIN)
- new net: D8.2 (A), JP1.2 (B)
- new net: NeoD4.1 (DOUT), NeoD5.3 (DIN)
- new net: NeoD3.1 (DOUT), NeoD4.3 (DIN)
- new net: NeoD14.1 (DOUT), NeoD15.3 (DIN)
- new net: NeoD13.1 (DOUT), NeoD14.3 (DIN)
- new net: D8.1 (K), NeoD1.3 (DIN), Q5.1 (D), R1.2
- new net: NeoD2.1 (DOUT), NeoD3.3 (DIN)
- new net: NeoD1.1 (DOUT), NeoD2.3 (DIN)
- new net: NeoD10.3 (DIN), NeoD9.1 (DOUT)
- new net: NeoD17.1 (DOUT), NeoD18.3 (DIN)
- new net: D11.2 (A), JP4.2 (B)
- new net: NeoD22.1 (DOUT), NeoD23.3 (DIN)
- new net: NeoD21.1 (DOUT), NeoD22.3 (DIN)
- new net: NeoD27.1 (DOUT), NeoD28.3 (DIN)
- new net: NeoD5.1 (DOUT), NeoD6.3 (DIN)
- new net: NeoD6.1 (DOUT), NeoD7.3 (DIN)
- new net: D10.1 (K), NeoD21.3 (DIN), Q7.1 (D), R18.2
- new net: D10.2 (A), JP3.2 (B)
- new net: D9.2 (A), JP2.2 (B)
- new net: NeoD7.1 (DOUT), NeoD8.3 (DIN)
- new net: NeoD8.1 (DOUT), NeoD9.3 (DIN)
- new net: NeoD11.1 (DOUT), NeoD12.3 (DIN)
- new net: NeoD12.1 (DOUT), NeoD13.3 (DIN)
- new net GPIO_NP_BOARD: JP4.1 (A), Q8.3 (S), U3.2 (GPIO0)
- no-connect marks 21 -> 19
Other:
- note added: "Neopixel WS2812B-2020"
- note removed: "Heater 1"
- note removed: "Heater 2"
- moved on the sheet: D4, D5, D6, D7, Q3, Q4, R19, R20
