File: hardware_kicad/filament_dryer.kicad_sch (KiCad schematic)
At the start: 71 parts, among them J4 Peristaltic Pump, U1 Pico, U2 H/T Filament, U3 H/T Filament, U4 DS18B20Z, U5 H/T Silicagel

Commit message: board outline cleaned up
Parts:
- removed R12: 10k, Resistor_SMD:R_0402_1005Metric_Pad0.72x0.64mm_HandSolder, symbol 00_project_library:R
- added D5: W, 00_project_library:LED_0603_1608Metric, symbol 00_project_library:LED
- added D8: R, 00_project_library:LED_0603_1608Metric, symbol 00_project_library:LED
- added D9: G, 00_project_library:LED_0603_1608Metric, symbol 00_project_library:LED
- added Elmwood-D139-2: Thermal Fulse, 00_project_library:Thermal Fuse (R_Axial_Power_L25.0mm_W6.4mm_P27.94mm), symbol 00_project_library:Thermal_Fuse
- added R10, R11, R9: 470R, Resistor_SMD:R_0402_1005Metric_Pad0.72x0.64mm_HandSolder, symbol 00_project_library:R
- added USER_BUTTON1: USER, 00_project_library:SW_TS-1187A-B-A-B, symbol 00_project_library:SW_MEC_5E
- R15: value 2k -> 4k7
- R3: value 10k -> 470R
- R6: value 10k -> 10K
- TP11: value HT_AMBIENT_SCL -> I2C0_SCL
- TP6: value HT_AMBIENT_SCA -> I2C0_SCA
- U3: value H/T Filament -> H/T Ambient
- renumbered U1 to P1, U2 to U1, U5 to U2
Connections:
- net +3V3: no longer R3.1, U2.2 (ADDR)
- net +5V: now also Elmwood-D139-2.1; no longer PowerR1.1, PowerR10.1, PowerR11.1, PowerR12.1, PowerR13.1, PowerR14.1, PowerR15.1, PowerR16.1, PowerR17.1, PowerR18.1, PowerR19.1, PowerR2.1, PowerR20.1, PowerR21.1, PowerR22.1, PowerR23.1, PowerR24.1, PowerR3.1, PowerR4.1, PowerR5.1, PowerR6.1, PowerR7.1, PowerR8.1, PowerR9.1
- net GND: now also U2.2 (ADDR), R10.1, R11.1, R9.1, USER_BUTTON1.1, USER_BUTTON1.2
- net HT_AMBIENT_SCL: no longer R8.2, U3.4 (SCL)
- net HT_AMBIENT_SDA: no longer R7.2, U3.1 (SDA)
- net at U1.6 (~{RESET}): no longer R3.2
- net at U3.6 (~{RESET}): no longer R6.2
- net at J4.2: now also R3.2
- net HT_FILAMENT_SCL renamed I2C1_SCL
- net HT_FILAMENT_SDA renamed I2C1_SDA
- new net: Elmwood-D139-2.2, PowerR1.1, PowerR10.1, PowerR11.1, PowerR12.1, PowerR13.1, PowerR14.1, PowerR15.1, PowerR16.1, PowerR17.1, PowerR18.1, PowerR19.1, PowerR2.1, PowerR20.1, PowerR21.1, PowerR22.1, PowerR23.1, PowerR24.1, PowerR3.1, PowerR4.1, PowerR5.1, PowerR6.1, PowerR7.1, PowerR8.1, PowerR9.1
- new net: D9.1 (K), R11.2
- new net: D8.1 (K), R10.2
- new net: D5.1 (K), R9.2
- new net GPIO_PUMP_ENABLE: R3.1
- new net GPIO_USER_BUTTON: R6.2, USER_BUTTON1.3 (K), USER_BUTTON1.4 (A)
- new net GPIO_USER_LED_GREEN: D9.2 (A)
- new net GPIO_USER_LED_RED: D8.2 (A)
- new net GPIO_USER_LED_WHITE: D5.2 (A)
- new net I2C0_SCL: R8.2, U3.4 (SCL)
- new net I2C0_SDA: R7.2, U3.1 (SDA)
- no-connect marks 4 -> 6
Other:
- note added: "H/T Ambient spare I2C0 0x44"
- note added: "USER LED"
- note added: "User Button"
- note removed: "H/T Ambient spare I2C0 0x45"
- moved on the sheet: C1, C2, C20, R22, R5, R8
