File: hardware_kicad/filament_dryer.kicad_sch (KiCad schematic)
At the start: 77 parts, among them J4 Peristaltic Pump, P1 Pico, U1 H/T Filament, U2 H/T Silicagel, U3 H/T Ambient, U4 DS18B20Z

Commit message: fet renumbered
Connections:
- net GND: now also FanQ1.2 (S), FanQ2.2 (S), PowerQ1.2 (S), PowerQ2.2 (S); no longer FanQ1.3 (S), FanQ2.3 (S), PowerQ1.3 (S), PowerQ2.3 (S)
- net GPIO_FAN_AMBIENT: now also FanQ1.1 (G); no longer FanQ1.2 (G)
- net GPIO_FAN_SILICAGEL: now also FanQ2.1 (G); no longer FanQ2.2 (G)
- net GPIO_HEATER_A: now also PowerQ1.1 (G); no longer PowerQ1.2 (G)
- net GPIO_HEATER_B: now also PowerQ2.1 (G); no longer PowerQ2.2 (G)
- net HEATER-A: now also PowerQ1.3 (D); no longer PowerQ1.1 (D)
- net HEATER-B: now also PowerQ2.3 (D); no longer PowerQ2.1 (D)
- net at D1.2 (A), TP8.1: now also FanQ1.3 (D); no longer FanQ1.1 (D)
- net at D2.2 (A), TP10.1: now also FanQ2.3 (D); no longer FanQ2.1 (D)
Changed lines of the file:
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@@
     (stroke (width 0) (type default))
   )
+  (wire (pts (xy 35.56 63.5) (xy 50.8 63.5))
+    (stroke (width 0) (type default))
+  )
   (wire (pts (xy 227.33 58.42) (xy 229.87 58.42))
     (stroke (width 0) (type solid))
@@
     (stroke (width 0) (type default))
   )
+  (wire (pts (xy 35.56 60.96) (xy 50.8 60.96))
+    (stroke (width 0) (type default))
+  )
   (wire (pts (xy 97.79 76.2) (xy 86.36 76.2))
     (stroke (width 0) (type default))
@@
     (effects (font (size 1.27 1.27)) (justify right bottom))
   )
-  (label "GPIO_PUMP_STEP" (at 50.8 60.96 180) (fields_autoplaced)
+  (label "GPIO_PUMP_STEP" (at 35.56 60.96 180) (fields_autoplaced)
     (effects (font (size 1.27 1.27)) (justify right bottom))
   )
@@
     (effects (font (size 1.27 1.27) italic) (justify right bottom))
   )
-  (label "GPIO_PUMP_ENABLE" (at 50.8 63.5 180) (fields_autoplaced)
+  (label "GPIO_PUMP_ENABLE" (at 35.56 63.5 180) (fields_autoplaced)
     (effects (font (size 1.27 1.27)) (justify right bottom))
   )
@@
       (effects (font (size 1.27 1.27)) hide)
     )
-    (property "Sim.Pins" "1=G 2=S 3=D" (at 163.83 118.11 0)
-      (effects (font (size 1.27 1.27)) hide)
-    )
     (property "JLC Part" "C143946" (at 170.18 105.41 0)
       (effects (font (size 1.27 1.27)) (justify left))
@@
       (effects (font (size 1.27 1.27)) hide)
     )
-    (property "Sim.Pins" "1=G 2=S 3=D" (at 52.07 207.01 0)
-      (effects (font (size 1.27 1.27)) hide)
-    )
     (property "JLC Part" "C143946" (at 58.42 194.31 0)
       (effects (font (size 1.27 1.27)) (justify left))
@@
       (effects (font (size 1.27 1.27)) hide)
     )
-    (property "Sim.Pins" "1=G 2=S 3=D" (at 162.56 156.21 0)
-      (effects (font (size 1.27 1.27)) hide)
-    )
     (property "JLC Part" "C143946" (at 168.91 143.51 0)
       (effects (font (size 1.27 1.27)) (justify left))
@@
       (effects (font (size 1.27 1.27)) hide)
     )
-    (property "Sim.Pins" "1=G 2=S 3=D" (at 134.62 205.74 0)
-      (effects (font (size 1.27 1.27)) hide)
-    )

Commit message: v1.0
Parts:
- removed R6: 10K, Resistor_SMD:R_0402_1005Metric_Pad0.72x0.64mm_HandSolder, symbol 00_project_library:R
- C1, C2: JLC (none) -> C96446
- C20: JCL (none) -> C96446
- D3: value Power_LED_1 -> HEATER_A
- D4: value Power_LED_2 -> HEATER_B
- TP11: value HT_AMBIENT_SCL -> HT_SPARE_SCL
- TP2: value HT_AMBIENT_GND -> HT_SPARE_GND
- TP3: value HT_AMBIENT_3V3 -> HT_SPARE_3V3
- TP6: value HT_AMBIENT_SDA -> HT_SPARE_SDA
- U2: value H/T Silicagel -> H/T Heater
Connections:
- net GPIO_HEATER_A: now also P1.10 (GPIO7); no longer P1.4 (GPIO2)
- net GPIO_HEATER_B: now also P1.4 (GPIO2); no longer P1.5 (GPIO3)
- net GPIO_PUMP_ENABLE: now also P1.20 (GPIO15); no longer P1.2 (GPIO1)
- net GPIO_PUMP_STEP: now also P1.19 (GPIO14); no longer P1.1 (GPIO0)
Other:
- note added: "H/T Heater I2C1 0x44"
- note added: "H/T spare I2C0 0x44"
- note removed: "H/T Ambient spare I2C0 0x44"
- note removed: "H/T Silicagel I2C1 0x44"
- moved on the sheet: C1, USER_BUTTON1

Commit message: v1.1 PCB
Parts:
- removed J4: Peristaltic Pump, 00_project_library:grove_vert_holes, symbol 00_project_library:grove_vert_holes
- removed R15: 4k7, Resistor_SMD:R_0402_1005Metric_Pad0.72x0.64mm_HandSolder, symbol 00_project_library:R
- removed R22, R3: 470R, Resistor_SMD:R_0402_1005Metric_Pad0.72x0.64mm_HandSolder, symbol 00_project_library:R
- removed TP11: HT_SPARE_SCL, TestPoint:TestPoint_Pad_D3.0mm, symbol Connector:TestPoint
- removed TP3: HT_SPARE_3V3, TestPoint:TestPoint_Pad_D3.0mm, symbol Connector:TestPoint
- removed TP6: HT_SPARE_SDA, TestPoint:TestPoint_Pad_D3.0mm, symbol Connector:TestPoint
- removed U4: DS18B20Z, 00_project_library:SOIC-8_3.9x4.9mm_P1.27mm, symbol 00_project_library:DS18B20Z
- added D10: WHITE, 00_project_library:LED_0603_1608Metric, symbol 00_project_library:LED
- added D11: General Purpose Diode, 00_project_library:D_SMA, symbol 00_project_library:GeneralPurposeDiode
- added FanQ3: NMOS, 00_project_library:SOT-23, symbol 00_project_library:NMOS
- added R6: 470R, Resistor_SMD:R_0402_1005Metric_Pad0.72x0.64mm_HandSolder, symbol 00_project_library:R
- added TP1: B+, TestPoint:TestPoint_Pad_D3.0mm, symbol Connector:TestPoint
- D6: value FAN_1 -> RED
- D7: value FAN_2 -> WHITE; JLC C2286 -> C2290
- TP10: value FAN_SILICAGEL_GND -> S-
- TP2: value HT_SPARE_GND -> B-
- TP7: value FAN_AMBIENT_5V -> A+
- TP8: value FAN_AMBIENT_GND -> A-
- TP9: value FAN_SILICAGEL_5V -> S+
Connections:
- net +5V: now also D11.1 (K), TP1.1
- net GND: now also FanQ3.2 (S), R6.2; no longer TP2.1
- net GPIO_FAN_AMBIENT: now also P1.7 (GPIO5)
- net GPIO_FAN_BOX: now reaches P1.6 (GPIO4)
- net GPIO_FAN_BOX: now also D10.2 (A), FanQ3.1 (G)
- net GPIO_FAN_SILICAGEL renamed GPIO_FAN_FILAMENT
- net GPIO_PUMP_ENABLE: no longer names the net of P1.20 (GPIO15)
- net GPIO_PUMP_STEP: no longer names the net of P1.19 (GPIO14)
- net T_HEATING_1WIRE: no longer names the net of P1.34 (GPIO28_ADC2)
- new net: D10.1 (K), R6.1
- new net: D11.2 (A), FanQ3.3 (D), TP2.1
- no-connect marks 26 -> 24
Other:
- note added: "Fan Box"
- note added: "Fan Filament"
- note removed: "Fan Silicagel"
- note removed: "H/T spare I2C0 0x44"
- note removed: "Peristaltic Pump"
- note removed: "Temperature"
