File: hardware_kicad/filament_dryer.kicad_pcb (KiCad board)
At the start: 2 copper layers, 70 x 107 mm, 77 parts, among them J4 Peristaltic Pump, P1 Pico, U1 H/T Filament, U2 H/T Silicagel, U3 H/T Ambient, U4 DS18B20Z

Commit message: layouting
Parts:
- added R1: 470R, Resistor_SMD:R_0402_1005Metric_Pad0.72x0.64mm_HandSolder, F.Cu at (191.6, 124.8)
- TP11: value I2C0_SCL -> HT_AMBIENT_SCL
- TP6: value I2C0_SCA -> HT_AMBIENT_SDA
- moved C2 151.5 mm to (151.7, 121.6)
- moved FanQ2 135.0 mm to (77.8, 136.5), turned to -90 degrees
- moved R15 101.0 mm to (101.5, 114.4)
- moved R8 73.5 mm to (71.5, 87.5)
- moved R7 72.8 mm to (68.7, 87.5), turned to 180 degrees
- moved PowerQ1 71.6 mm to (131.4, 79.2)
- moved PowerQ2 71.5 mm to (131.3, 85.3)
- moved J4 64.3 mm to (130.4, 63.5)
- moved R9 50.3 mm to (92.1, 155.1)
- moved C20 50.3 mm to (96.0, 112.1), turned to 90 degrees
- moved R10 50.0 mm to (92.1, 157.8)
- moved R11 49.9 mm to (92.0, 160.4)
- moved R6 40.4 mm to (103.0, 153.1), turned to 180 degrees
- moved U1 28.8 mm to (151.5, 69.0)
- moved TP9 28.6 mm to (69.5, 135.8)
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Connections:
- net /HT_AMBIENT_SCL renamed /i2C0_SCL
- net Net-(PowerQ1-D) renamed /HEATER-A
- net Net-(PowerQ2-D) renamed /HEATER-B
- Elmwood-D139-2 pad 1: +5V -> /5V-Fuse
- Elmwood-D139-2 pad 2: Net-(Elmwood-D139-2-Pad2) -> +5V
- P1 pad 21: unconnected-(P1-GPIO16-Pad21) -> /I2C0_SDA
- P1 pad 22: unconnected-(P1-GPIO17-Pad22) -> /I2C0_SCL
- P1 pad 24: unconnected-(P1-GPIO18-Pad24) -> /GPIO_FAN_SILICAGEL
- P1 pad 25: unconnected-(P1-GPIO19-Pad25) -> /GPIO_USER_LED_WHITE
- P1 pad 26: unconnected-(P1-GPIO20-Pad26) -> /GPIO_USER_LED_RED
- P1 pad 27: unconnected-(P1-GPIO21-Pad27) -> /GPIO_USER_LED_GREEN
- P1 pad 29: unconnected-(P1-GPIO22-Pad29) -> /GPIO_USER_BUTTON
- P1 pad 31: unconnected-(P1-GPIO26_ADC0-Pad31) -> /I2C1_SDA
- P1 pad 32: unconnected-(P1-GPIO27_ADC1-Pad32) -> /I2C1_SCL
- P1 pad 34: unconnected-(P1-GPIO28_ADC2-Pad34) -> /T_HEATING_1WIRE
- PowerR1 pad 1: Net-(Elmwood-D139-2-Pad2) -> /5V-Fuse
- PowerR10 pad 1: Net-(Elmwood-D139-2-Pad2) -> /5V-Fuse
- PowerR11 pad 1: Net-(Elmwood-D139-2-Pad2) -> /5V-Fuse
- PowerR12 pad 1: Net-(Elmwood-D139-2-Pad2) -> /5V-Fuse
- PowerR13 pad 1: Net-(Elmwood-D139-2-Pad2) -> /5V-Fuse
- PowerR14 pad 1: Net-(Elmwood-D139-2-Pad2) -> /5V-Fuse
- PowerR15 pad 1: Net-(Elmwood-D139-2-Pad2) -> /5V-Fuse
- PowerR16 pad 1: Net-(Elmwood-D139-2-Pad2) -> /5V-Fuse
- PowerR17 pad 1: Net-(Elmwood-D139-2-Pad2) -> /5V-Fuse
- PowerR18 pad 1: Net-(Elmwood-D139-2-Pad2) -> /5V-Fuse
- PowerR19 pad 1: Net-(Elmwood-D139-2-Pad2) -> /5V-Fuse
- PowerR2 pad 1: Net-(Elmwood-D139-2-Pad2) -> /5V-Fuse
- PowerR20 pad 1: Net-(Elmwood-D139-2-Pad2) -> /5V-Fuse
- PowerR21 pad 1: Net-(Elmwood-D139-2-Pad2) -> /5V-Fuse
- PowerR22 pad 1: Net-(Elmwood-D139-2-Pad2) -> /5V-Fuse
- PowerR23 pad 1: Net-(Elmwood-D139-2-Pad2) -> /5V-Fuse
- PowerR24 pad 1: Net-(Elmwood-D139-2-Pad2) -> /5V-Fuse
- PowerR3 pad 1: Net-(Elmwood-D139-2-Pad2) -> /5V-Fuse
- PowerR4 pad 1: Net-(Elmwood-D139-2-Pad2) -> /5V-Fuse
- PowerR5 pad 1: Net-(Elmwood-D139-2-Pad2) -> /5V-Fuse
- PowerR6 pad 1: Net-(Elmwood-D139-2-Pad2) -> /5V-Fuse
- PowerR7 pad 1: Net-(Elmwood-D139-2-Pad2) -> /5V-Fuse
- PowerR8 pad 1: Net-(Elmwood-D139-2-Pad2) -> /5V-Fuse
- PowerR9 pad 1: Net-(Elmwood-D139-2-Pad2) -> /5V-Fuse
- TP6 pad 1: /HT_AMBIENT_SDA -> /I2C0_SDA
Routing:
- net +3V3: track 68.3 -> 224.0 mm, vias 2 -> 5
- net /GPIO_USER_BUTTON: track 0.00 -> 102.7 mm, vias 0 -> 2
- net /I2C0_SCL: track 0.00 -> 98.5 mm, vias 0 -> 2
- net /I2C0_SDA: track 0.00 -> 97.6 mm, vias 0 -> 2
- net /GPIO_USER_LED_GREEN: track 0.00 -> 94.7 mm, vias 0 -> 2
- net /GPIO_USER_LED_RED: track 0.00 -> 91.3 mm, vias 0 -> 2
- net /GPIO_USER_LED_WHITE: track 0.00 -> 84.8 mm, vias 0 -> 2
- net /I2C1_SDA: track 0.00 -> 70.8 mm
- net /T_HEATING_1WIRE: track 0.00 -> 64.1 mm, vias 0 -> 4
- net Net-(D2-A): track 6.10 -> 69.6 mm
- net /GPIO_FAN_SILICAGEL: track 0.00 -> 62.8 mm, vias 0 -> 2
- net /I2C1_SCL: track 0.00 -> 61.8 mm, vias 0 -> 2
- net /HEATER-A: track 0.00 -> 56.4 mm, vias 0 -> 13
- net /HEATER-B: track 0.00 -> 55.1 mm, vias 0 -> 13
- net GND: track 63.1 -> 23.5 mm
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- added copper zone on F.Cu, net /5V-Fuse
- added copper zone on B.Cu, net /HEATER-A
- added copper zone on B.Cu, net /HEATER-B
- added copper zone on F.Cu, net GND
- removed copper zone on F.Cu, net +5V
Other:
- board size 70 x 107 mm -> 70 x 112 mm
- board text added: "locked"
- board text removed: "${TITLE} ${ISSUE_DATE} ${REVISION}"
